File: Amiga-Stereo-Digitizer/Amiga-Stereo-Digitizer.kicad_pcb (KiCad board)
At the start: 2 copper layers, 71.4 x 53.1 mm, 39 parts, among them IC1 LM555CM, IC2 ADC0809CCV_NOPB, IC4 MC74HC14ADTR2G, J0 L717SDB25P1ACH4F, J1 OS-Select, J2 RCJ-043, J3 RCJ-042, U3 LM324DR

Commit message: Add files via upload
Other:
- board text added: "rev.1"
- board text removed: "rev.0"

Commit message: Add files via upload
Parts:
- removed G***: LOGO, SamacSys_Parts:stereo-logo
- removed REF**: MountingHole_2.5mm_Pad_Via, MountingHole:MountingHole_2.5mm_Pad_Via
- C1, C3: value 47nF -> 10nF
- C2, C4: value 1uF -> 22uF
- C6: footprint Capacitor_SMD:CP_Elec_4x5.8 -> Capacitor_SMD:C_0805_2012Metric
Routing:
- net VCC: track 124.1 -> 124.8 mm
Other:
- board text added: "rev.2"
- board text removed: "rev.1"

Commit message: Add files via upload
Parts:
- added REF**: MountingHole_2.5mm_Pad, MountingHole:MountingHole_2.5mm_Pad, F.Cu at (144.0, 90.7)
